File: led_mapper_850/single_net.kicad_sch (KiCad schematic)
At the start: 530 parts, among them J1 Conn_02x12_Top_Bottom

Commit message: rename single net schematic
Parts:
- renumbered D471 to D1000, D472 to D1001, D473 to D1002, D474 to D1003, D475 to D1004, D476 to D1005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

Commit message: clean up front connector wires
Parts:
- renumbered D530 to D1, D539 to D10, D629 to D100, D630 to D101, D631 to D102, D632 to D103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
