File: led_mapper_850/kicad_project/led_mapper_850.kicad_sch (KiCad schematic)
At the start: 1 part, among them J1 Conn_02x12_Top_Bottom

Commit message: add fabrication outputs for previewing PCBA quote
Parts:
- J1: LCSC Part # (none) -> C19268781
Changed lines of the file:
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@@
 			)
 		)
-		(property "LCSC PN" ""
+		(property "LCSC Part #" "C19268781"
 			(at 107.95 171.45 0)
 			(effects
