File: led_mapper_850/kicad_project/single_net_reverse_cols.kicad_sch (KiCad schematic)
At the start: 529 parts

Commit message: rework row vias & front row shorts
Connections:
- net P1: now also D?.1 (K), D?.1 (K), D?.1 (K), D?.1 (K), D?.1 (K), D?.1 (K), D?.1 (K), D?.1 (K), D?.1 (K), D?.1 (K), D?.1 (K), D?.1 (K), D?.1 (K), D?.1 (K), D?.1 (K), D?.1 (K), D?.1 (K), D?.1 (K), D?.1 (K), D?.1 (K), D?.1 (K), D?.1 (K), D?.1 (K)
- net P10: now also D?.1 (K), D?.1 (K), D?.1 (K), D?.1 (K), D?.1 (K), D?.1 (K), D?.1 (K), D?.1 (K), D?.1 (K), D?.1 (K), D?.1 (K), D?.1 (K), D?.1 (K), D?.1 (K), D?.1 (K), D?.1 (K), D?.1 (K), D?.1 (K), D?.1 (K), D?.1 (K), D?.1 (K), D?.1 (K), D?.1 (K); no longer D?.1 (K), D?.1 (K), D?.1 (K), D?.1 (K), D?.1 (K), D?.1 (K), D?.1 (K), D?.1 (K), D?.1 (K), D?.1 (K), D?.1 (K), D?.1 (K), D?.1 (K), D?.1 (K), D?.1 (K), D?.1 (K), D?.1 (K), D?.1 (K), D?.1 (K), D?.1 (K), D?.1 (K), D?.1 (K), D?.1 (K)
- net P11: now also D?.1 (K), D?.1 (K), D?.1 (K), D?.1 (K), D?.1 (K), D?.1 (K), D?.1 (K), D?.1 (K), D?.1 (K), D?.1 (K), D?.1 (K), D?.1 (K), D?.1 (K), D?.1 (K), D?.1 (K), D?.1 (K), D?.1 (K), D?.1 (K), D?.1 (K), D?.1 (K), D?.1 (K), D?.1 (K), D?.1 (K); no longer D?.1 (K), D?.1 (K), D?.1 (K), D?.1 (K), D?.1 (K), D?.1 (K), D?.1 (K), D?.1 (K), D?.1 (K), D?.1 (K), D?.1 (K), D?.1 (K), D?.1 (K), D?.1 (K), D?.1 (K), D?.1 (K), D?.1 (K), D?.1 (K), D?.1 (K), D?.1 (K), D?.1 (K), D?.1 (K), D?.1 (K)
- net P12: now also D?.1 (K), D?.1 (K), D?.1 (K), D?.1 (K), D?.1 (K), D?.1 (K), D?.1 (K), D?.1 (K), D?.1 (K), D?.1 (K), D?.1 (K), D?.1 (K), D?.1 (K), D?.1 (K), D?.1 (K), D?.1 (K), D?.1 (K), D?.1 (K), D?.1 (K), D?.1 (K), D?.1 (K), D?.1 (K), D?.1 (K); no longer D?.1 (K), D?.1 (K), D?.1 (K), D?.1 (K), D?.1 (K), D?.1 (K), D?.1 (K), D?.1 (K), D?.1 (K), D?.1 (K), D?.1 (K), D?.1 (K), D?.1 (K), D?.1 (K), D?.1 (K), D?.1 (K), D?.1 (K), D?.1 (K), D?.1 (K), D?.1 (K), D?.1 (K), D?.1 (K), D?.1 (K)
- net P13: now also D?.1 (K), D?.1 (K), D?.1 (K), D?.1 (K), D?.1 (K), D?.1 (K), D?.1 (K), D?.1 (K), D?.1 (K), D?.1 (K), D?.1 (K), D?.1 (K), D?.1 (K), D?.1 (K), D?.1 (K), D?.1 (K), D?.1 (K), D?.1 (K), D?.1 (K), D?.1 (K), D?.1 (K), D?.1 (K), D?.1 (K); no longer D?.1 (K), D?.1 (K), D?.1 (K), D?.1 (K), D?.1 (K), D?.1 (K), D?.1 (K), D?.1 (K), D?.1 (K), D?.1 (K), D?.1 (K), D?.1 (K), D?.1 (K), D?.1 (K), D?.1 (K), D?.1 (K), D?.1 (K), D?.1 (K), D?.1 (K), D?.1 (K), D?.1 (K), D?.1 (K), D?.1 (K)
- net P14: now also D?.1 (K), D?.1 (K), D?.1 (K), D?.1 (K), D?.1 (K), D?.1 (K), D?.1 (K), D?.1 (K), D?.1 (K), D?.1 (K), D?.1 (K), D?.1 (K), D?.1 (K), D?.1 (K), D?.1 (K), D?.1 (K), D?.1 (K), D?.1 (K), D?.1 (K), D?.1 (K), D?.1 (K), D?.1 (K), D?.1 (K); no longer D?.1 (K), D?.1 (K), D?.1 (K), D?.1 (K), D?.1 (K), D?.1 (K), D?.1 (K), D?.1 (K), D?.1 (K), D?.1 (K), D?.1 (K), D?.1 (K), D?.1 (K), D?.1 (K), D?.1 (K), D?.1 (K), D?.1 (K), D?.1 (K), D?.1 (K), D?.1 (K), D?.1 (K), D?.1 (K), D?.1 (K)
- net P15: now also D?.1 (K), D?.1 (K), D?.1 (K), D?.1 (K), D?.1 (K), D?.1 (K), D?.1 (K), D?.1 (K), D?.1 (K), D?.1 (K), D?.1 (K), D?.1 (K), D?.1 (K), D?.1 (K), D?.1 (K), D?.1 (K), D?.1 (K), D?.1 (K), D?.1 (K), D?.1 (K), D?.1 (K), D?.1 (K), D?.1 (K); no longer D?.1 (K), D?.1 (K), D?.1 (K), D?.1 (K), D?.1 (K), D?.1 (K), D?.1 (K), D?.1 (K), D?.1 (K), D?.1 (K), D?.1 (K), D?.1 (K), D?.1 (K), D?.1 (K), D?.1 (K), D?.1 (K), D?.1 (K), D?.1 (K), D?.1 (K), D?.1 (K), D?.1 (K), D?.1 (K), D?.1 (K)
- net P16: now also D?.1 (K), D?.1 (K), D?.1 (K), D?.1 (K), D?.1 (K), D?.1 (K), D?.1 (K), D?.1 (K), D?.1 (K), D?.1 (K), D?.1 (K), D?.1 (K), D?.1 (K), D?.1 (K), D?.1 (K), D?.1 (K), D?.1 (K), D?.1 (K), D?.1 (K), D?.1 (K), D?.1 (K), D?.1 (K), D?.1 (K); no longer D?.1 (K), D?.1 (K), D?.1 (K), D?.1 (K), D?.1 (K), D?.1 (K), D?.1 (K), D?.1 (K), D?.1 (K), D?.1 (K), D?.1 (K), D?.1 (K), D?.1 (K), D?.1 (K), D?.1 (K), D?.1 (K), D?.1 (K), D?.1 (K), D?.1 (K), D?.1 (K), D?.1 (K), D?.1 (K), D?.1 (K)
- net P17: now also D?.1 (K), D?.1 (K), D?.1 (K), D?.1 (K), D?.1 (K), D?.1 (K), D?.1 (K), D?.1 (K), D?.1 (K), D?.1 (K), D?.1 (K), D?.1 (K), D?.1 (K), D?.1 (K), D?.1 (K), D?.1 (K), D?.1 (K), D?.1 (K), D?.1 (K), D?.1 (K), D?.1 (K), D?.1 (K), D?.1 (K); no longer D?.1 (K), D?.1 (K), D?.1 (K), D?.1 (K), D?.1 (K), D?.1 (K), D?.1 (K), D?.1 (K), D?.1 (K), D?.1 (K), D?.1 (K), D?.1 (K), D?.1 (K), D?.1 (K), D?.1 (K), D?.1 (K), D?.1 (K), D?.1 (K), D?.1 (K), D?.1 (K), D?.1 (K), D?.1 (K), D?.1 (K)
- net P18: now also D?.1 (K), D?.1 (K), D?.1 (K), D?.1 (K), D?.1 (K), D?.1 (K), D?.1 (K), D?.1 (K), D?.1 (K), D?.1 (K), D?.1 (K), D?.1 (K), D?.1 (K), D?.1 (K), D?.1 (K), D?.1 (K), D?.1 (K), D?.1 (K), D?.1 (K), D?.1 (K), D?.1 (K), D?.1 (K), D?.1 (K); no longer D?.1 (K), D?.1 (K), D?.1 (K), D?.1 (K), D?.1 (K), D?.1 (K), D?.1 (K), D?.1 (K), D?.1 (K), D?.1 (K), D?.1 (K), D?.1 (K), D?.1 (K), D?.1 (K), D?.1 (K), D?.1 (K), D?.1 (K), D?.1 (K), D?.1 (K), D?.1 (K), D?.1 (K), D?.1 (K), D?.1 (K)
- net P19: now also D?.1 (K), D?.1 (K), D?.1 (K), D?.1 (K), D?.1 (K), D?.1 (K), D?.1 (K), D?.1 (K), D?.1 (K), D?.1 (K), D?.1 (K), D?.1 (K), D?.1 (K), D?.1 (K), D?.1 (K), D?.1 (K), D?.1 (K), D?.1 (K), D?.1 (K), D?.1 (K), D?.1 (K), D?.1 (K), D?.1 (K); no longer D?.1 (K), D?.1 (K), D?.1 (K), D?.1 (K), D?.1 (K), D?.1 (K), D?.1 (K), D?.1 (K), D?.1 (K), D?.1 (K), D?.1 (K), D?.1 (K), D?.1 (K), D?.1 (K), D?.1 (K), D?.1 (K), D?.1 (K), D?.1 (K), D?.1 (K), D?.1 (K), D?.1 (K), D?.1 (K), D?.1 (K)
- net P2: now also D?.1 (K), D?.1 (K), D?.1 (K), D?.1 (K), D?.1 (K), D?.1 (K), D?.1 (K), D?.1 (K), D?.1 (K), D?.1 (K), D?.1 (K), D?.1 (K), D?.1 (K), D?.1 (K), D?.1 (K), D?.1 (K), D?.1 (K), D?.1 (K), D?.1 (K), D?.1 (K), D?.1 (K), D?.1 (K), D?.1 (K); no longer D?.1 (K), D?.1 (K), D?.1 (K), D?.1 (K), D?.1 (K), D?.1 (K), D?.1 (K), D?.1 (K), D?.1 (K), D?.1 (K), D?.1 (K), D?.1 (K), D?.1 (K), D?.1 (K), D?.1 (K), D?.1 (K), D?.1 (K), D?.1 (K), D?.1 (K), D?.1 (K), D?.1 (K), D?.1 (K), D?.1 (K)
- net P20: now also D?.1 (K), D?.1 (K), D?.1 (K), D?.1 (K), D?.1 (K), D?.1 (K), D?.1 (K), D?.1 (K), D?.1 (K), D?.1 (K), D?.1 (K), D?.1 (K), D?.1 (K), D?.1 (K), D?.1 (K), D?.1 (K), D?.1 (K), D?.1 (K), D?.1 (K), D?.1 (K), D?.1 (K), D?.1 (K), D?.1 (K); no longer D?.1 (K), D?.1 (K), D?.1 (K), D?.1 (K), D?.1 (K), D?.1 (K), D?.1 (K), D?.1 (K), D?.1 (K), D?.1 (K), D?.1 (K), D?.1 (K), D?.1 (K), D?.1 (K), D?.1 (K), D?.1 (K), D?.1 (K), D?.1 (K), D?.1 (K), D?.1 (K), D?.1 (K), D?.1 (K), D?.1 (K)
- net P21: now also D?.1 (K), D?.1 (K), D?.1 (K), D?.1 (K), D?.1 (K), D?.1 (K), D?.1 (K), D?.1 (K), D?.1 (K), D?.1 (K), D?.1 (K), D?.1 (K), D?.1 (K), D?.1 (K), D?.1 (K), D?.1 (K), D?.1 (K), D?.1 (K), D?.1 (K), D?.1 (K), D?.1 (K), D?.1 (K), D?.1 (K); no longer D?.1 (K), D?.1 (K), D?.1 (K), D?.1 (K), D?.1 (K), D?.1 (K), D?.1 (K), D?.1 (K), D?.1 (K), D?.1 (K), D?.1 (K), D?.1 (K), D?.1 (K), D?.1 (K), D?.1 (K), D?.1 (K), D?.1 (K), D?.1 (K), D?.1 (K), D?.1 (K), D?.1 (K), D?.1 (K), D?.1 (K)
- net P22: now also D?.1 (K), D?.1 (K), D?.1 (K), D?.1 (K), D?.1 (K), D?.1 (K), D?.1 (K), D?.1 (K), D?.1 (K), D?.1 (K), D?.1 (K), D?.1 (K), D?.1 (K), D?.1 (K), D?.1 (K), D?.1 (K), D?.1 (K), D?.1 (K), D?.1 (K), D?.1 (K), D?.1 (K), D?.1 (K), D?.1 (K); no longer D?.1 (K), D?.1 (K), D?.1 (K), D?.1 (K), D?.1 (K), D?.1 (K), D?.1 (K), D?.1 (K), D?.1 (K), D?.1 (K), D?.1 (K), D?.1 (K), D?.1 (K), D?.1 (K), D?.1 (K), D?.1 (K), D?.1 (K), D?.1 (K), D?.1 (K), D?.1 (K), D?.1 (K), D?.1 (K), D?.1 (K)
- net P23: now also D?.1 (K), D?.1 (K), D?.1 (K), D?.1 (K), D?.1 (K), D?.1 (K), D?.1 (K), D?.1 (K), D?.1 (K), D?.1 (K), D?.1 (K), D?.1 (K), D?.1 (K), D?.1 (K), D?.1 (K), D?.1 (K), D?.1 (K), D?.1 (K), D?.1 (K), D?.1 (K), D?.1 (K), D?.1 (K), D?.1 (K); no longer D?.1 (K), D?.1 (K), D?.1 (K), D?.1 (K), D?.1 (K), D?.1 (K), D?.1 (K), D?.1 (K), D?.1 (K), D?.1 (K), D?.1 (K), D?.1 (K), D?.1 (K), D?.1 (K), D?.1 (K), D?.1 (K), D?.1 (K), D?.1 (K), D?.1 (K), D?.1 (K), D?.1 (K), D?.1 (K), D?.1 (K)
- net P24: no longer D?.1 (K), D?.1 (K), D?.1 (K), D?.1 (K), D?.1 (K), D?.1 (K), D?.1 (K), D?.1 (K), D?.1 (K), D?.1 (K), D?.1 (K), D?.1 (K), D?.1 (K), D?.1 (K), D?.1 (K), D?.1 (K), D?.1 (K), D?.1 (K), D?.1 (K), D?.1 (K), D?.1 (K), D?.1 (K), D?.1 (K)
- net P3: now also D?.1 (K), D?.1 (K), D?.1 (K), D?.1 (K), D?.1 (K), D?.1 (K), D?.1 (K), D?.1 (K), D?.1 (K), D?.1 (K), D?.1 (K), D?.1 (K), D?.1 (K), D?.1 (K), D?.1 (K), D?.1 (K), D?.1 (K), D?.1 (K), D?.1 (K), D?.1 (K), D?.1 (K), D?.1 (K), D?.1 (K); no longer D?.1 (K), D?.1 (K), D?.1 (K), D?.1 (K), D?.1 (K), D?.1 (K), D?.1 (K), D?.1 (K), D?.1 (K), D?.1 (K), D?.1 (K), D?.1 (K), D?.1 (K), D?.1 (K), D?.1 (K), D?.1 (K), D?.1 (K), D?.1 (K), D?.1 (K), D?.1 (K), D?.1 (K), D?.1 (K), D?.1 (K)
- net P4: now also D?.1 (K), D?.1 (K), D?.1 (K), D?.1 (K), D?.1 (K), D?.1 (K), D?.1 (K), D?.1 (K), D?.1 (K), D?.1 (K), D?.1 (K), D?.1 (K), D?.1 (K), D?.1 (K), D?.1 (K), D?.1 (K), D?.1 (K), D?.1 (K), D?.1 (K), D?.1 (K), D?.1 (K), D?.1 (K), D?.1 (K); no longer D?.1 (K), D?.1 (K), D?.1 (K), D?.1 (K), D?.1 (K), D?.1 (K), D?.1 (K), D?.1 (K), D?.1 (K), D?.1 (K), D?.1 (K), D?.1 (K), D?.1 (K), D?.1 (K), D?.1 (K), D?.1 (K), D?.1 (K), D?.1 (K), D?.1 (K), D?.1 (K), D?.1 (K), D?.1 (K), D?.1 (K)
- net P5: now also D?.1 (K), D?.1 (K), D?.1 (K), D?.1 (K), D?.1 (K), D?.1 (K), D?.1 (K), D?.1 (K), D?.1 (K), D?.1 (K), D?.1 (K), D?.1 (K), D?.1 (K), D?.1 (K), D?.1 (K), D?.1 (K), D?.1 (K), D?.1 (K), D?.1 (K), D?.1 (K), D?.1 (K), D?.1 (K), D?.1 (K); no longer D?.1 (K), D?.1 (K), D?.1 (K), D?.1 (K), D?.1 (K), D?.1 (K), D?.1 (K), D?.1 (K), D?.1 (K), D?.1 (K), D?.1 (K), D?.1 (K), D?.1 (K), D?.1 (K), D?.1 (K), D?.1 (K), D?.1 (K), D?.1 (K), D?.1 (K), D?.1 (K), D?.1 (K), D?.1 (K), D?.1 (K)
- net P6: now also D?.1 (K), D?.1 (K), D?.1 (K), D?.1 (K), D?.1 (K), D?.1 (K), D?.1 (K), D?.1 (K), D?.1 (K), D?.1 (K), D?.1 (K), D?.1 (K), D?.1 (K), D?.1 (K), D?.1 (K), D?.1 (K), D?.1 (K), D?.1 (K), D?.1 (K), D?.1 (K), D?.1 (K), D?.1 (K), D?.1 (K); no longer D?.1 (K), D?.1 (K), D?.1 (K), D?.1 (K), D?.1 (K), D?.1 (K), D?.1 (K), D?.1 (K), D?.1 (K), D?.1 (K), D?.1 (K), D?.1 (K), D?.1 (K), D?.1 (K), D?.1 (K), D?.1 (K), D?.1 (K), D?.1 (K), D?.1 (K), D?.1 (K), D?.1 (K), D?.1 (K), D?.1 (K)
- net P7: now also D?.1 (K), D?.1 (K), D?.1 (K), D?.1 (K), D?.1 (K), D?.1 (K), D?.1 (K), D?.1 (K), D?.1 (K), D?.1 (K), D?.1 (K), D?.1 (K), D?.1 (K), D?.1 (K), D?.1 (K), D?.1 (K), D?.1 (K), D?.1 (K), D?.1 (K), D?.1 (K), D?.1 (K), D?.1 (K), D?.1 (K); no longer D?.1 (K), D?.1 (K), D?.1 (K), D?.1 (K), D?.1 (K), D?.1 (K), D?.1 (K), D?.1 (K), D?.1 (K), D?.1 (K), D?.1 (K), D?.1 (K), D?.1 (K), D?.1 (K), D?.1 (K), D?.1 (K), D?.1 (K), D?.1 (K), D?.1 (K), D?.1 (K), D?.1 (K), D?.1 (K), D?.1 (K)
- net P8: now also D?.1 (K), D?.1 (K), D?.1 (K), D?.1 (K), D?.1 (K), D?.1 (K), D?.1 (K), D?.1 (K), D?.1 (K), D?.1 (K), D?.1 (K), D?.1 (K), D?.1 (K), D?.1 (K), D?.1 (K), D?.1 (K), D?.1 (K), D?.1 (K), D?.1 (K), D?.1 (K), D?.1 (K), D?.1 (K), D?.1 (K); no longer D?.1 (K), D?.1 (K), D?.1 (K), D?.1 (K), D?.1 (K), D?.1 (K), D?.1 (K), D?.1 (K), D?.1 (K), D?.1 (K), D?.1 (K), D?.1 (K), D?.1 (K), D?.1 (K), D?.1 (K), D?.1 (K), D?.1 (K), D?.1 (K), D?.1 (K), D?.1 (K), D?.1 (K), D?.1 (K), D?.1 (K)
- net P9: now also D?.1 (K), D?.1 (K), D?.1 (K), D?.1 (K), D?.1 (K), D?.1 (K), D?.1 (K), D?.1 (K), D?.1 (K), D?.1 (K), D?.1 (K), D?.1 (K), D?.1 (K), D?.1 (K), D?.1 (K), D?.1 (K), D?.1 (K), D?.1 (K), D?.1 (K), D?.1 (K), D?.1 (K), D?.1 (K), D?.1 (K); no longer D?.1 (K), D?.1 (K), D?.1 (K), D?.1 (K), D?.1 (K), D?.1 (K), D?.1 (K), D?.1 (K), D?.1 (K), D?.1 (K), D?.1 (K), D?.1 (K), D?.1 (K), D?.1 (K), D?.1 (K), D?.1 (K), D?.1 (K), D?.1 (K), D?.1 (K), D?.1 (K), D?.1 (K), D?.1 (K), D?.1 (K)

Commit message: add led part number - XINGLIGHT Red 0201
Parts:
- D? (x529): LCSC PN (none) -> C3646923

Commit message: add fabrication outputs for previewing PCBA quote
Parts:
- D? (x529): LCSC PN C3646923 -> (none); LCSC Part # (none) -> C3646923

Commit message: fix critical schematic error - wrong pins
Connections:
- net P01 is gone; now on net P1: D?.2 (A), D?.2 (A), D?.2 (A), D?.2 (A), D?.2 (A), D?.2 (A), D?.2 (A), D?.2 (A), D?.2 (A), D?.2 (A), D?.2 (A)
- net P02 is gone; now on net P2: D?.2 (A), D?.2 (A), D?.2 (A), D?.2 (A), D?.2 (A), D?.2 (A), D?.2 (A), D?.2 (A), D?.2 (A), D?.2 (A), D?.2 (A)
- net P03 is gone; now on net P3: D?.2 (A), D?.2 (A), D?.2 (A), D?.2 (A), D?.2 (A), D?.2 (A), D?.2 (A), D?.2 (A), D?.2 (A), D?.2 (A), D?.2 (A)
- net P04 is gone; now on net P4: D?.2 (A), D?.2 (A), D?.2 (A), D?.2 (A), D?.2 (A), D?.2 (A), D?.2 (A), D?.2 (A), D?.2 (A), D?.2 (A), D?.2 (A)
- net P05 is gone; now on net P5: D?.2 (A), D?.2 (A), D?.2 (A), D?.2 (A), D?.2 (A), D?.2 (A), D?.2 (A), D?.2 (A), D?.2 (A), D?.2 (A), D?.2 (A)
- net P06 is gone; now on net P6: D?.2 (A), D?.2 (A), D?.2 (A), D?.2 (A), D?.2 (A), D?.2 (A), D?.2 (A), D?.2 (A), D?.2 (A), D?.2 (A), D?.2 (A)
- net P07 is gone; now on net P7: D?.2 (A), D?.2 (A), D?.2 (A), D?.2 (A), D?.2 (A), D?.2 (A), D?.2 (A), D?.2 (A), D?.2 (A), D?.2 (A), D?.2 (A)
- net P08 is gone; now on net P8: D?.2 (A), D?.2 (A), D?.2 (A), D?.2 (A), D?.2 (A), D?.2 (A), D?.2 (A), D?.2 (A), D?.2 (A), D?.2 (A), D?.2 (A)
- net P09 is gone; now on net P9: D?.2 (A), D?.2 (A), D?.2 (A), D?.2 (A), D?.2 (A), D?.2 (A), D?.2 (A), D?.2 (A), D?.2 (A), D?.2 (A), D?.2 (A)
Changed lines of the file:
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@@
 		)
 	)
-	(label "P03"
+	(label "P3"
 		(at 189.23 20.32 0)
 		(effects
@@
 		)
 	)
-	(label "P04"
+	(label "P4"
 		(at 181.61 20.32 0)
 		(effects
@@
 		)
 	)
-	(label "P07"
+	(label "P7"
 		(at 158.75 20.32 0)
 		(effects
@@
 		)
 	)
-	(label "P08"
+	(label "P8"
 		(at 151.13 20.32 0)
 		(effects
@@
 		)
 	)
-	(label "P05"
+	(label "P5"
 		(at 173.99 20.32 0)
 		(effects
@@
 		)
 	)
-	(label "P09"
+	(label "P9"
 		(at 143.51 20.32 0)
 		(effects
@@
 		)
 	)
-	(label "P02"
+	(label "P2"
 		(at 196.85 20.32 0)
 		(effects
@@
 		)
 	)
-	(label "P01"
+	(label "P1"
 		(at 204.47 20.32 0)
 		(effects
@@
 		)
 	)
-	(label "P06"
+	(label "P6"
 		(at 166.37 20.32 0)
 		(effects

Commit message: fix network issues (pin name mismatch)
Parts:
- removed D?: LED, LED_SMD:LED_0201_0603Metric, symbol Device:LED_45deg
- added D552: LED, LED_SMD:LED_0201_0603Metric, symbol Device:LED_45deg
Connections:
- net P1: now also D552.1 (K)
- net P2: now also D552.2 (A)
Changed lines of the file:
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@@
 	)
 	(junction
+		(at 196.85 31.75)
+		(diameter 0)
+		(color 0 0 0 0)
+	)
+	(junction
 		(at 90.17 54.61)
 		(diameter 0)
@@
 	)
 	(junction
-		(at 196.85 31.75)
-		(diameter 0)
-		(color 0 0 0 0)
-	)
-	(junction
 		(at 64.77 87.63)
 		(diameter 0)
@@
 	(wire
 		(pts
-			(xy 196.85 31.75) (xy 196.85 46.99)
+			(xy 196.85 20.32) (xy 196.85 31.75)
 		)
 		(stroke
@@
 	(wire
 		(pts
+			(xy 196.85 31.75) (xy 196.85 46.99)
+		)
+		(stroke
+			(width 0)
+			(type default)
+		)
+	)
+	(wire
+		(pts
 			(xy 392.43 77.47) (xy 392.43 85.09)
 		)
@@
 	(wire
 		(pts
-			(xy 196.85 20.32) (xy 196.85 31.75)
-		)
-		(stroke
-			(width 0)
-			(type default)
-		)
-	)
-	(wire
-		(pts
 			(xy 59.69 85.09) (xy 59.69 92.71)
 		)
@@
 	(symbol
 		(lib_id "Device:LED_45deg")
-		(at 199.39 29.21 90)
-		(unit 1)
-		(exclude_from_sim no)
-		(in_bom yes)
-		(on_board yes)
-		(dnp no)
-		(property "Reference" "D?"
-			(at 196.85 27.686 90)
-			(effects
-				(font
-					(size 1.27 1.27)
-				)
-				(justify right)
-			)
-		)
-		(property "Value" "LED"
-			(at 199.898 30.988 90)
-			(effects
-				(font
-					(size 1.27 1.27)
-				)
-				(justify right)
-				(hide yes)
-			)
-		)
-		(property "Footprint" "LED_SMD:LED_0201_0603Metric"
-			(at 199.39 29.21 0)
-			(effects
-				(font
-					(size 1.27 1.27)
-				)
-				(hide yes)
-			)
-		)
-		(property "Datasheet" "~"
-			(at 199.39 29.21 0)
-			(effects
-				(font
-					(size 1.27 1.27)
-				)
-				(hide yes)
-			)
-		)
-		(property "Description" "Light emitting diode, rotated by 45°"
-			(at 199.39 29.21 0)
-			(effects
-				(font
-					(size 1.27 1.27)
-				)
-				(hide yes)
-			)
-		)
-		(property "LCSC Part #" "C3646923"
-			(at 199.39 29.21 0)
-			(effects
-				(font
-					(size 1.27 1.27)
-				)
-				(hide yes)
-			)
-		)
-		(pin "1"
-		)
-		(pin "2"
-		)
-		(instances
-			(project "single_net_reverse_cols"
-				(path "/47ee292d-1c66-48a5-a287-ef8b334ccd42"
-					(reference "D?")
-					(unit 1)
-				)
-			)
-			(project "led_mapper_850"
-				(path "/51b7e780-688f-494d-9172-4437a593740a/acdf1064-22a7-45b0-b045-023df4437ef1"
-					(reference "D1610")
-					(unit 1)
-				)
-				(path "/51b7e780-688f-494d-9172-4437a593740a/d9c8edf6-0db8-4a05-9e19-e51ea97e1f56"
-					(reference "D552")
-					(unit 1)
-				)
-			)
-		)
-	)
-	(symbol
-		(lib_id "Device:LED_45deg")
 		(at 295.91 59.69 90)
 		(unit 1)
@@
 					(unit 1)
 				)
+			)
+		)
+	)
+	(symbol
+		(lib_id "Device:LED_45deg")
+		(at 199.39 29.21 90)
+		(unit 1)
+		(exclude_from_sim no)
+		(in_bom yes)
+		(on_board yes)
+		(dnp no)
+		(property "Reference" "D552"
+			(at 196.85 27.686 90)
+			(effects
+				(font
+					(size 1.27 1.27)
+				)
+				(justify right)
+			)
+		)
+		(property "Value" "LED"
+			(at 199.898 30.988 90)
+			(effects
+				(font
+					(size 1.27 1.27)
+				)
+				(justify right)
+				(hide yes)
+			)
+		)
+		(property "Footprint" "LED_SMD:LED_0201_0603Metric"
+			(at 199.39 29.21 0)
+			(effects
+				(font
+					(size 1.27 1.27)
+				)
+				(hide yes)
+			)
+		)
+		(property "Datasheet" "~"
+			(at 199.39 29.21 0)
+			(effects
+				(font
+					(size 1.27 1.27)
+				)
+				(hide yes)
+			)
+		)
+		(property "Description" "Light emitting diode, rotated by 45°"
+			(at 199.39 29.21 0)
+			(effects
+				(font
+					(size 1.27 1.27)
+				)
+				(hide yes)
+			)
+		)
+		(property "LCSC Part #" "C3646923"
+			(at 199.39 29.21 0)
+			(effects
+				(font
+					(size 1.27 1.27)
+				)
+				(hide yes)
+			)
+		)
+		(pin "1"
+		)
+		(pin "2"
+		)
+		(instances
+			(project "led_mapper_850"
+				(path "/51b7e780-688f-494d-9172-4437a593740a/acdf1064-22a7-45b0-b045-023df4437ef1"
+					(reference "D1610")
+					(unit 1)
+				)
+				(path "/51b7e780-688f-494d-9172-4437a593740a/d9c8edf6-0db8-4a05-9e19-e51ea97e1f56"
+					(reference "D552")
+					(unit 1)
+				)
