File: led_mapper_850/mirrored_rhombus/single_net_reverse_cols.kicad_sch (KiCad schematic)
At the start: 529 parts

Commit message: mirror rhombus
Parts:
- renumbered D552 to D1610
Changed lines of the file:
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@@
 		(on_board yes)
 		(dnp no)
-		(property "Reference" "D552"
+		(property "Reference" "D1610"
 			(at 196.85 27.686 90)
 			(effects

Commit message: Sync changes: update holes to 2.2mm, change footprint to match datasheet
Parts:
- D1610, D? (x528): footprint LED_SMD:LED_0201_0603Metric -> ccatlib:LED_0201_0603Metric_XINGLIGHT
