File: led_mapper_850/mirrored_rhombus/single_net.kicad_sch (KiCad schematic)
At the start: 529 parts

Commit message: missed file - schematic
Parts:
- D1, D10, D100, D101, D102, D103, D104, D105, D106, D107, D108, D109, D11, D110, D111, D112, D113, D114, D115, D116, D117, D118, D119, D12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: footprint LED_SMD:LED_0201_0603Metric -> ccatlib:LED_0201_0603Metric_XINGLIGHT
